File: PCR/PCR/PCR.kicad_pcb (KiCad board)
At the start: 2 copper layers, 7 parts, among them Q1 BC413, U1 TemperatureSensor, U2 Arduino, U3 TemperatureSensor

Commit message: Revised Schematic/PCB for PCR
Parts:
- removed U1: TemperatureSensor, Wire_Connections_Bridges:WireConnection_2.50mmDrill
- added U4: Amplifier, PCR:thermo_amp, F.Cu at (191.8, 83.8)
- D1: footprint Diodes_ThroughHole:Diode_P600_Horizontal -> Resistors_ThroughHole:R_Axial_DIN0207_L6.3mm_D2.5mm_P7.62mm_Horizontal
- Q1: footprint TO_SOT_Packages_THT:TO-92_Inline_Wide -> Pin_Headers:Pin_Header_Straight_1x03_Pitch2.54mm
- R1: footprint Resistors_ThroughHole:Resistor_Horizontal_RM30mm -> Resistors_ThroughHole:R_Axial_DIN0207_L6.3mm_D2.5mm_P7.62mm_Horizontal
- R2: footprint Wire_Connections_Bridges:WireConnection_2.50mmDrill_LargePad -> Pin_Headers:Pin_Header_Straight_1x02_Pitch2.54mm
- U2: footprint Wire_Connections_Bridges:WireConnection_2.50mmDrill_LargePad -> PCR:arduino_pin_header
- U3: value TemperatureSensor -> Amplifier; footprint Wire_Connections_Bridges:WireConnection_2.50mmDrill -> PCR:thermo_amp
- moved R1 85.2 mm to (161.3, 116.8), turned to 90 degrees
- moved D1 84.1 mm to (185.4, 109.2), turned to 270 degrees
- moved U2 44.6 mm to (193.0, 102.9), turned to 270 degrees
- moved Q1 36.9 mm to (174.0, 114.3), turned to 180 degrees
- moved U3 27.7 mm to (166.4, 83.8)
- moved R2 20.9 mm to (196.8, 109.2)
Connections:
- Q1 pad 3: +24V -> Net-(Q1-Pad3)
- R1 pad 2: +24V -> Net-(Q1-Pad3)
- U3 pad 1: (no net) -> Net-(U2-Pad13)
- U3 pad 2: (no net) -> Net-(U3-Pad2)
Routing:
- net Net-(U2-Pad17): track 0.00 -> 41.0 mm
- net Net-(U2-Pad13): track 0.00 -> 35.8 mm
- net Net-(D1-Pad2): track 0.00 -> 31.7 mm
- net Net-(Q1-Pad2): track 0.00 -> 30.7 mm
- net Net-(D1-Pad1): track 0.00 -> 25.0 mm
- net Net-(Q1-Pad3): track 0.00 -> 23.9 mm
- net Net-(U2-Pad4): track 0.00 -> 12.5 mm
- net Net-(U2-Pad5): track 0.00 -> 11.8 mm
- net Net-(U2-Pad6): track 0.00 -> 11.8 mm
- net Net-(U2-Pad11): track 0.00 -> 10.7 mm
- net Net-(U2-Pad12): track 0.00 -> 10.7 mm
- net Net-(U2-Pad10): track 0.00 -> 10.7 mm
Other:
- board outline added: 50.8 x 50.8 mm
- net class 24V added: clearance 0.2, trace_width 1.016, via_dia 0.6, via_drill 0.4

Commit message: Version 2 of the PCB
Parts:
- added CON1: BARREL_JACK, Connect:BARREL_JACK, F.Cu at (190.5, 114.3)
- added G***: LOGO, PCR:cidar_logo_adjusted_4, B.Cu at (179.7, 78.7)
- Q1: value BC413 -> BUZ11
- U2: footprint PCR:arduino_pin_header -> PCR:Arduino_Pin_Header_1x10
- moved U2 29.2 mm to (163.8, 101.6), turned to 90 degrees
- moved R2 16.6 mm to (180.3, 108.0), turned to 90 degrees
- moved R1 10.5 mm to (163.8, 106.7), turned to 270 degrees
- moved D1 9.16 mm to (177.8, 114.3), turned to 0 degrees
- moved Q1 5.24 mm to (172.7, 109.2), turned to 0 degrees
- moved U4 1.80 mm to (190.5, 85.1)
- moved U3 1.80 mm to (167.6, 85.1)
Connections:
- D1 pad 2: Net-(D1-Pad2) -> Net-(CON1-Pad2)
- Q1 pad 1: Net-(D1-Pad1) -> Net-(Q1-Pad1)
- Q1 pad 2: Net-(Q1-Pad2) -> Net-(D1-Pad1)
- Q1 pad 3: Net-(Q1-Pad3) -> Net-(CON1-Pad1)
- R1 pad 1: Net-(Q1-Pad2) -> Net-(Q1-Pad1)
- R1 pad 2: Net-(Q1-Pad3) -> Net-(CON1-Pad1)
- R2 pad 2: Net-(D1-Pad2) -> Net-(CON1-Pad2)
- U2 pad 16: Net-(Q1-Pad3) -> Net-(CON1-Pad1)
- U2 pad 3: Net-(Q1-Pad2) -> Net-(Q1-Pad1)
Routing:
- net Net-(D1-Pad2): track 31.7 -> 0.00 mm
- net Net-(Q1-Pad2): track 30.7 -> 0.00 mm
- net Net-(Q1-Pad1): track 0.00 -> 25.0 mm
- net Net-(CON1-Pad2): track 0.00 -> 24.8 mm
- net Net-(Q1-Pad3): track 23.9 -> 0.00 mm
- net Net-(D1-Pad1): track 25.0 -> 13.2 mm
- net Net-(U2-Pad5): track 11.8 -> 19.4 mm
- net Net-(U2-Pad4): track 12.5 -> 20.1 mm
- net Net-(U2-Pad6): track 11.8 -> 18.6 mm
- net Net-(U2-Pad17): track 41.0 -> 34.6 mm
- net Net-(U2-Pad11): track 10.7 -> 7.11 mm
- net Net-(U2-Pad12): track 10.7 -> 7.11 mm
- net Net-(U2-Pad10): track 10.7 -> 7.11 mm
- net Net-(U2-Pad13): track 35.8 -> 38.5 mm
- added copper zone on B.Cu, net Net-(CON1-Pad1)
Other:
- net class 3.3V added: clearance 0.2, trace_width 1.016, via_dia 0.6, via_drill 0.4
- net class Analog_Ground added: clearance 0.2, trace_width 1.016, via_dia 0.6, via_drill 0.4
- net class Default: trace_width 0.25 -> 0.508
- board text added: "Designed By Alex Nero"
- board text added: "Vulcan PCR v 2.0"
