File: PCR/PCR/PCR.sch (KiCad schematic (older format))
At the start: 7 parts, among them Q1 BC413, U1 TemperatureSensor, U2 Arduino, U3 TemperatureSensor

Commit message: New PCB data
Parts:
- removed U1, U3: TemperatureSensor, Pin_Headers:Pin_Header_Straight_1x03, symbol TemperatureSensor
- removed U2: Arduino, Pin_Headers:Pin_Header_Straight_1x06, symbol Arduino
- added TC? (x2): Thermocouple, symbol Thermocouple
- added U?: Arduino, symbol Arduino
- added U? (x2): Amplifier, symbol Amplifier
- added U?: Fan, symbol Fan
Connections:
- wire segments 30 -> 57
Other:
- moved on the sheet: D1, Q1, R1, R2

Commit message: Revised Schematic/PCB for PCR
Parts:
- removed U?: Fan, symbol Fan
- D1: footprint Diodes_ThroughHole:Diode_P600_Horizontal -> Resistors_ThroughHole:R_Axial_DIN0207_L6.3mm_D2.5mm_P7.62mm_Horizontal
- Q1: footprint TO_SOT_Packages_THT:TO-92_Inline_Wide -> Pin_Headers:Pin_Header_Straight_1x03_Pitch2.54mm
- R1: footprint Resistors_ThroughHole:Resistor_Horizontal_RM30mm -> Resistors_ThroughHole:R_Axial_DIN0207_L6.3mm_D2.5mm_P7.62mm_Horizontal
- R2: footprint Wire_Connections_Bridges:WireConnection_2.50mmDrill_LargePad -> Pin_Headers:Pin_Header_Straight_1x02_Pitch2.54mm
- U2: renamed from U?; footprint (none) -> PCR:arduino_pin_header
- U3, U4: renamed from U?; footprint (none) -> PCR:thermo_amp
- gave numbers to parts that had none: 2
Connections:
- net labels removed: +24V, Earth
- wire segments 57 -> 55
Other:
- moved on the sheet: TC1, TC2
Changed lines of the file:
@@
 $EndDescr
-$Comp
-L Earth #PWR02
-U 1 1 5840802F
-P 5250 6100
-F 0 "#PWR02" H 5250 5850 50  0001 C CNN
-F 1 "Earth" H 5250 5950 50  0001 C CNN
-F 2 "" H 5250 6100 50  0000 C CNN
-F 3 "" H 5250 6100 50  0000 C CNN
-	1    5250 6100
-	1    0    0    -1
-$EndComp
-$Comp
-L +24V #PWR03
-U 1 1 58408091
-P 6850 5650
-F 0 "#PWR03" H 6850 5500 50  0001 C CNN
-F 1 "+24V" H 6850 5790 50  0000 C CNN
-F 2 "" H 6850 5650 50  0000 C CNN
-F 3 "" H 6850 5650 50  0000 C CNN
-	1    6850 5650
-	1    0    0    -1
-$EndComp
 $Comp
 L BC413 Q1
@@
 F 0 "Q1" H 6050 5075 50  0000 L CNN
 F 1 "BC413" H 6050 5000 50  0000 L CNN
-F 2 "TO_SOT_Packages_THT:TO-92_Inline_Wide" H 6050 4925 50  0001 L CIN
+F 2 "Pin_Headers:Pin_Header_Straight_1x03_Pitch2.54mm" H 6050 4925 50  0001 L CIN
 F 3 "" H 5850 5000 50  0000 L CNN
 	1    5850 5000
@@
 F 0 "R2" V 7130 4950 50  0000 C CNN
 F 1 "Nichrome Wire" V 7050 4950 50  0000 C CNN
-F 2 "Wire_Connections_Bridges:WireConnection_2.50mmDrill_LargePad" V 6980 4950 50  0001 C CNN
+F 2 "Pin_Headers:Pin_Header_Straight_1x02_Pitch2.54mm" V 6980 4950 50  0001 C CNN
 F 3 "" H 7050 4950 50  0000 C CNN
 	1    7050 4950
@@
 F 0 "D1" H 6750 5100 50  0000 C CNN
 F 1 "D" H 6750 4900 50  0000 C CNN
-F 2 "Diodes_ThroughHole:Diode_P600_Horizontal" H 6750 5000 50  0001 C CNN
+F 2 "Resistors_ThroughHole:R_Axial_DIN0207_L6.3mm_D2.5mm_P7.62mm_Horizontal" H 6750 5000 50  0001 C CNN
 F 3 "" H 6750 5000 50  0000 C CNN
 	1    6750 5000
@@
 F 0 "R1" V 5580 5650 50  0000 C CNN
 F 1 "R" V 5500 5650 50  0000 C CNN
-F 2 "Resistors_ThroughHole:Resistor_Horizontal_RM30mm" V 5430 5650 50  0001 C CNN
+F 2 "Resistors_ThroughHole:R_Axial_DIN0207_L6.3mm_D2.5mm_P7.62mm_Horizontal" V 5430 5650 50  0001 C CNN
 F 3 "" H 5500 5650 50  0000 C CNN
 	1    5500 5650
@@
 $EndComp
 $Comp
-L Arduino U?
+L Arduino U2
 U 1 1 58C090EE
 P 5300 3800
-F 0 "U?" H 5450 3650 60  0000 C CNN
+F 0 "U2" H 5450 3650 60  0000 C CNN
 F 1 "Arduino" H 5450 4000 60  0000 C CNN
-F 2 "" H 5400 3200 60  0001 C CNN
+F 2 "PCR:arduino_pin_header" H 5400 3200 60  0001 C CNN
 F 3 "" H 5400 3200 60  0001 C CNN
 	1    5300 3800
@@
 $EndComp
 $Comp
-L Amplifier U?
+L Amplifier U3
 U 1 1 58C20272
 P 7450 3300
-F 0 "U?" H 7350 3550 60  0001 C CNN
+F 0 "U3" H 7350 3550 60  0001 C CNN
 F 1 "Amplifier" H 7350 3700 60  0000 C CNN
-F 2 "" H 7350 3700 60  0001 C CNN
+F 2 "PCR:thermo_amp" H 7350 3700 60  0001 C CNN
 F 3 "" H 7350 3700 60  0001 C CNN
 	1    7450 3300
@@
 $EndComp
 $Comp
-L Amplifier U?
+L Amplifier U4
 U 1 1 58C20290
 P 7950 4600
-F 0 "U?" H 7850 4850 60  0001 C CNN
+F 0 "U4" H 7850 4850 60  0001 C CNN
 F 1 "Amplifier" H 7850 5000 60  0000 C CNN
-F 2 "" H 7850 5000 60  0001 C CNN
+F 2 "PCR:thermo_amp" H 7850 5000 60  0001 C CNN
 F 3 "" H 7850 5000 60  0001 C CNN
 	1    7950 4600
@@
 $EndComp
 $Comp
-L Fan U?
-U 1 1 58C204F8
-P 3850 3750
-F 0 "U?" H 3850 3700 60  0000 C CNN
-F 1 "Fan" H 3850 3850 60  0000 C CNN
-F 2 "" H 3850 3850 60  0001 C CNN
-F 3 "" H 3850 3850 60  0001 C CNN
-	1    3850 3750
-	1    0    0    -1
-$EndComp
-Wire Wire Line
-	5950 5200 5950 6100
-Wire Wire Line
-	5250 6100 6850 6100
+L Thermocouple TC1
+U 1 1 58C1FAB1
+P 8400 3125
+F 0 "TC1" H 8280 3275 50  0000 C CNN
+F 1 "Thermocouple" H 8200 2965 50  0000 L CNN
+F 2 "" H 7825 3175 50  0001 C CNN
+F 3 "" H 7825 3175 50  0001 C CNN
+	1    8400 3125
+	-1   0    0    -1
+$EndComp
+$Comp
+L Thermocouple TC2
+U 1 1 58C1FAFF
+P 8950 4425
+F 0 "TC2" H 8830 4575 50  0000 C CNN
+F 1 "Thermocouple" H 8750 4265 50  0000 L CNN
+F 2 "" H 8375 4475 50  0001 C CNN
+F 3 "" H 8375 4475 50  0001 C CNN
+	1    8950 4425
+	-1   0    0    -1
+$EndComp
+Wire Wire Line
+	5950 6100 5950 5200
+Wire Wire Line
+	4450 6100 5950 6100
 Wire Wire Line
 	5250 6100 5250 5800
 Connection ~ 5250 5800
 Wire Wire Line
-	6850 5550 6850 5150
+	6850 5550 6850 5550
+Wire Wire Line
+	6850 5150 6850 6325
 Wire Wire Line
 	6750 5150 7050 5150
@@
 	6900 4800 5950 4800
 Connection ~ 6900 4800
-Wire Wire Line
-	6850 6100 6850 5650
 Connection ~ 5950 6100
 Wire Wire Line
@@
 	6650 3400 6800 3400
 Wire Wire Line
-	4850 3500 4850 2550
+	4850 2550 4850 3525
 Wire Wire Line
 	4850 2550 7200 2550
@@
 	6100 2350 7800 2350
 Wire Wire Line
-	7450 2350 7450 2550
+	7425 2350 7425 2550
 Wire Wire Line
 	6100 4300 6700 4300
@@
 	6700 4700 7300 4700
 Wire Wire Line
-	6200 4150 6800 4150
+	6100 4150 6800 4150
 Wire Wire Line
 	6800 4150 6800 4500
@@
 	7800 2350 7800 3850
 Wire Wire Line
-	7800 3850 7950 3850
-Connection ~ 7450 2350
-Wire Wire Line
-	6100 3750 6300 3750
-Wire Wire Line
-	6300 3750 6300 2850
-Wire Wire Line
-	6300 2850 3850 2850
-Wire Wire Line
-	3850 4150 4450 4150
-Wire Wire Line
-	4450 4150 4450 3800
+	7800 3850 7925 3850
+Connection ~ 7425 2350
+Wire Wire Line
+	8350 4325 8850 4325
+Wire Wire Line
+	8850 4600 8350 4600
+Wire Wire Line
+	8850 4525 8850 4600
+Wire Wire Line
+	8300 3300 7850 3300
+Wire Wire Line
+	8300 3225 8300 3300
+Wire Wire Line
+	7850 3025 8300 3025
+Wire Wire Line
+	4450 6100 4450 3800
 Wire Wire Line
 	4450 3800 4850 3800
-Wire Wire Line
-	3850 2850 3850 3350
-$Comp
-L Thermocouple TC?
-U 1 1 58C1FAB1
-P 8400 3150
-F 0 "TC?" H 8280 3300 50  0000 C CNN
-F 1 "Thermocouple" H 8200 2990 50  0000 L CNN
-F 2 "" H 7825 3200 50  0001 C CNN
-F 3 "" H 7825 3200 50  0001 C CNN
-	1    8400 3150
-	-1   0    0    -1
-$EndComp
-$Comp
-L Thermocouple TC?
-U 1 1 58C1FAFF
-P 8950 4450
-F 0 "TC?" H 8830 4600 50  0000 C CNN
-F 1 "Thermocouple" H 8750 4290 50  0000 L CNN
-F 2 "" H 8375 4500 50  0001 C CNN
-F 3 "" H 8375 4500 50  0001 C CNN
-	1    8950 4450
-	-1   0    0    -1
-$EndComp
-Wire Wire Line
-	8350 4350 8850 4350
-Wire Wire Line
-	8350 4600 8850 4600
-Wire Wire Line
-	8850 4600 8850 4550
-Wire Wire Line
-	7850 3300 8300 3300
-Wire Wire Line
-	8300 3300 8300 3250
-Wire Wire Line
-	7850 3050 8300 3050
+Connection ~ 5250 6100
+Wire Wire Line
+	6850 6325 4200 6325
+Wire Wire Line
+	4200 6325 4200 3650
+Wire Wire Line
+	4200 3650 4850 3650
 $EndSCHEMATC

Commit message: Version 2 of the PCB
Parts:
- removed Q1: BC413, Pin_Headers:Pin_Header_Straight_1x03_Pitch2.54mm, symbol BC413
- added CON1: BARREL_JACK, Connect:BARREL_JACK, symbol BARREL_JACK
- added Q1: BUZ11, Pin_Headers:Pin_Header_Straight_1x03_Pitch2.54mm, symbol BUZ11
- U2: footprint PCR:arduino_pin_header -> PCR:Arduino_Pin_Header_1x10
Connections:
- wire segments 55 -> 46
- no-connect marks 0 -> 3
Other:
- moved on the sheet: R1, R2
Changed lines of the file:
@@
 $EndDescr
-$Comp
-L BC413 Q1
-U 1 1 58409174
-P 5850 5000
-F 0 "Q1" H 6050 5075 50  0000 L CNN
-F 1 "BC413" H 6050 5000 50  0000 L CNN
-F 2 "Pin_Headers:Pin_Header_Straight_1x03_Pitch2.54mm" H 6050 4925 50  0001 L CIN
-F 3 "" H 5850 5000 50  0000 L CNN
-	1    5850 5000
-	1    0    0    -1
-$EndComp
 $Comp
 L R R2
 U 1 1 584091EE
-P 7050 4950
-F 0 "R2" V 7130 4950 50  0000 C CNN
-F 1 "Nichrome Wire" V 7050 4950 50  0000 C CNN
-F 2 "Pin_Headers:Pin_Header_Straight_1x02_Pitch2.54mm" V 6980 4950 50  0001 C CNN
-F 3 "" H 7050 4950 50  0000 C CNN
-	1    7050 4950
+P 7200 4950
+F 0 "R2" V 7280 4950 50  0000 C CNN
+F 1 "Nichrome Wire" V 7200 4950 50  0000 C CNN
+F 2 "Pin_Headers:Pin_Header_Straight_1x02_Pitch2.54mm" V 7130 4950 50  0001 C CNN
+F 3 "" H 7200 4950 50  0000 C CNN
+	1    7200 4950
 	1    0    0    -1
 $EndComp
@@
 L R R1
 U 1 1 584099E6
-P 5500 5650
-F 0 "R1" V 5580 5650 50  0000 C CNN
-F 1 "R" V 5500 5650 50  0000 C CNN
-F 2 "Resistors_ThroughHole:R_Axial_DIN0207_L6.3mm_D2.5mm_P7.62mm_Horizontal" V 5430 5650 50  0001 C CNN
-F 3 "" H 5500 5650 50  0000 C CNN
-	1    5500 5650
+P 5500 5350
+F 0 "R1" V 5580 5350 50  0000 C CNN
+F 1 "R" V 5500 5350 50  0000 C CNN
+F 2 "Resistors_ThroughHole:R_Axial_DIN0207_L6.3mm_D2.5mm_P7.62mm_Horizontal" V 5430 5350 50  0001 C CNN
+F 3 "" H 5500 5350 50  0000 C CNN
+	1    5500 5350
 	1    0    0    -1
 $EndComp
@@
 F 0 "U2" H 5450 3650 60  0000 C CNN
 F 1 "Arduino" H 5450 4000 60  0000 C CNN
-F 2 "PCR:arduino_pin_header" H 5400 3200 60  0001 C CNN
+F 2 "PCR:Arduino_Pin_Header_1x10" H 5400 3200 60  0001 C CNN
 F 3 "" H 5400 3200 60  0001 C CNN
 	1    5300 3800
@@
 	-1   0    0    -1
 $EndComp
-Wire Wire Line
-	5950 6100 5950 5200
-Wire Wire Line
-	4450 6100 5950 6100
-Wire Wire Line
-	5250 6100 5250 5800
-Connection ~ 5250 5800
-Wire Wire Line
-	6850 5550 6850 5550
-Wire Wire Line
-	6850 5150 6850 6325
-Wire Wire Line
-	6750 5150 7050 5150
-Wire Wire Line
-	7050 5150 7050 5100
+$Comp
+L BARREL_JACK CON1
+U 1 1 58D83E36
+P 7800 5575
+F 0 "CON1" H 7800 5825 50  0000 C CNN
+F 1 "BARREL_JACK" H 7800 5375 50  0000 C CNN
+F 2 "Connect:BARREL_JACK" H 7800 5575 50  0001 C CNN
+F 3 "" H 7800 5575 50  0000 C CNN
+	1    7800 5575
+	-1   0    0    1
+$EndComp
+$Comp
+L BUZ11 Q1
+U 1 1 58D848BB
+P 5850 5000
+F 0 "Q1" H 6100 5075 50  0000 L CNN
+F 1 "BUZ11" H 6100 5000 50  0000 L CNN
+F 2 "Pin_Headers:Pin_Header_Straight_1x03_Pitch2.54mm" H 6100 4925 50  0000 L CIN
+F 3 "" H 5850 5000 50  0000 L CNN
+	1    5850 5000
+	1    0    0    -1
+$EndComp
+Wire Wire Line
+	4850 5675 7500 5675
+Wire Wire Line
+	4850 3950 4850 5675
+Wire Wire Line
+	6100 4650 6100 4450
+Wire Wire Line
+	5500 4650 6100 4650
+Wire Wire Line
+	5500 4650 5500 5200
+Wire Wire Line
+	5500 5050 5650 5050
+Wire Wire Line
+	6100 3300 6400 3300
+Wire Wire Line
+	6400 3300 6400 3000
+Wire Wire Line
+	6400 3000 6800 3000
+Wire Wire Line
+	6100 3450 6500 3450
+Wire Wire Line
+	6500 3450 6500 3200
+Wire Wire Line
+	6500 3200 6800 3200
+Wire Wire Line
+	6100 3600 6600 3600
+Wire Wire Line
+	6600 3600 6600 3400
+Wire Wire Line
+	6600 3400 6800 3400
+Wire Wire Line
+	4850 2550 4850 3525
+Wire Wire Line
+	4850 2550 7200 2550
+Wire Wire Line
+	6100 3100 6100 2350
+Wire Wire Line
+	6100 2350 7925 2350
+Wire Wire Line
+	7425 2350 7425 2550
+Wire Wire Line
+	6100 4300 6700 4300
+Wire Wire Line
+	6700 4300 6700 4700
+Wire Wire Line
+	6700 4700 7300 4700
+Wire Wire Line
+	6100 4150 6800 4150
+Wire Wire Line
+	6800 4150 6800 4500
+Wire Wire Line
+	6800 4500 7300 4500
+Wire Wire Line
+	6100 4000 6900 4000
+Wire Wire Line
+	6900 4000 6900 4300
+Wire Wire Line
+	6900 4300 7300 4300
+Wire Wire Line
+	6700 2550 6700 3850
+Wire Wire Line
+	6700 3850 7700 3850
+Connection ~ 6700 2550
+Wire Wire Line
+	7925 2350 7925 3850
+Connection ~ 7425 2350
+Wire Wire Line
+	8350 4325 8850 4325
+Wire Wire Line
+	8850 4600 8350 4600
+Wire Wire Line
+	8850 4525 8850 4600
+Wire Wire Line
+	8300 3300 7850 3300
+Wire Wire Line
+	8300 3225 8300 3300
+Wire Wire Line
+	7850 3025 8300 3025
+Wire Wire Line
+	6850 5475 7500 5475
+Wire Wire Line
+	5950 5675 5950 5200
+Connection ~ 5500 5050
 Connection ~ 6850 5150
 Wire Wire Line
+	6850 5150 6850 5475
+Wire Wire Line
+	6750 5150 7200 5150
+Wire Wire Line
+	5950 4800 7200 4800
+Wire Wire Line
 	6750 4850 6750 4800
-Wire Wire Line
-	6750 4800 7050 4800
-Wire Wire Line
-	6900 4800 5950 4800
-Connection ~ 6900 4800
-Connection ~ 5950 6100
-Wire Wire Line
-	4850 5800 5500 5800
-Wire Wire Line
-	4850 3950 4850 5800
-Wire Wire Line
-	6100 4450 6100 4650
-Wire Wire Line
-	6100 4650 5650 4650
-Wire Wire Line
-	5650 4650 5650 5000
-Wire Wire Line
-	5500 5500 5500 5000
-Wire Wire Line
-	5500 5000 5650 5000
-Wire Wire Line
-	6100 3300 6400 3300
-Wire Wire Line
-	6400 3300 6400 3000
-Wire Wire Line
-	6400 3000 6800 3000
-Wire Wire Line
-	6100 3450 6500 3450
-Wire Wire Line
-	6500 3450 6500 3200
-Wire Wire Line
-	6500 3200 6800 3200
-Wire Wire Line
-	6100 3600 6650 3600
-Wire Wire Line
-	6650 3600 6650 3400
-Wire Wire Line
-	6650 3400 6800 3400
-Wire Wire Line
-	4850 2550 4850 3525
-Wire Wire Line
-	4850 2550 7200 2550
-Wire Wire Line
-	6100 3100 6100 2350
-Wire Wire Line
-	6100 2350 7800 2350
-Wire Wire Line
-	7425 2350 7425 2550
-Wire Wire Line
-	6100 4300 6700 4300
-Wire Wire Line
-	6700 4300 6700 4700
-Wire Wire Line
-	6700 4700 7300 4700
-Wire Wire Line
-	6100 4150 6800 4150
-Wire Wire Line
-	6800 4150 6800 4500
-Wire Wire Line
-	6800 4500 7300 4500
-Wire Wire Line
-	6100 4000 6900 4000
-Wire Wire Line
-	6900 4000 6900 4300
-Wire Wire Line
-	6900 4300 7300 4300
-Wire Wire Line
-	6850 2550 6850 3850
-Wire Wire Line
-	6850 3850 7700 3850
-Connection ~ 6850 2550
-Wire Wire Line
-	7800 2350 7800 3850
-Wire Wire Line
-	7800 3850 7925 3850
-Connection ~ 7425 2350
-Wire Wire Line
-	8350 4325 8850 4325
-Wire Wire Line
-	8850 4600 8350 4600
-Wire Wire Line
-	8850 4525 8850 4600
-Wire Wire Line
-	8300 3300 7850 3300
-Wire Wire Line
-	8300 3225 8300 3300
-Wire Wire Line
-	7850 3025 8300 3025
-Wire Wire Line
-	4450 6100 4450 3800
-Wire Wire Line
-	4450 3800 4850 3800
-Connection ~ 5250 6100
-Wire Wire Line
-	6850 6325 4200 6325
-Wire Wire Line
-	4200 6325 4200 3650
-Wire Wire Line
-	4200 3650 4850 3650
+Connection ~ 6750 4800
+Wire Wire Line
+	7200 5150 7200 5100
+Connection ~ 5950 5675
+Wire Wire Line
+	5500 5500 5500 5675
+Connection ~ 5500 5675
+NoConn ~ 6100 3750
+NoConn ~ 8350 4750
+NoConn ~ 7850 3450
 $EndSCHEMATC
